Commit message: second commit

File: resources/mobile_manipulator/kortex/urdf/gen3_robotiq_2f_85_platform.urdf (robot description, URDF)
Before this commit: robot gen3_robotiq_2f_85_platform, 33 links, 32 joints
Links:
- added link attachment
- added link root
Joints:
- removed joint back_left_caster_joint
- removed joint back_left_turning_joint
- removed joint back_right_caster_joint
- removed joint back_right_turning_joint
- removed joint base_to_arm_joint
- removed joint front_left_caster_joint
- removed joint front_left_turning_joint
- removed joint front_right_caster_joint
- removed joint front_right_turning_link
- removed joint joint_1
- removed joint joint_2
- removed joint joint_3
- removed joint joint_4
- removed joint joint_5
- removed joint joint_6
- removed joint joint_7
- added joint arm_joint_1: type revolute, parent base_link, child shoulder_link, origin xyz=0 0 0.15643 rpy=3.1416 2.7629E-18 -4.9305E-36, axis 0 0 1, limit lower=-300 upper=300 effort=39 velocity=1.05
- added joint arm_joint_2: type revolute, parent shoulder_link, child half_arm_1_link, origin xyz=0 0.005375 -0.12838 rpy=1.5708 2.1343E-17 -1.1102E-16, axis 0 0 1, limit lower=-2.24 upper=2.24 effort=39 velocity=1.05
- added joint arm_joint_3: type revolute, parent half_arm_1_link, child half_arm_2_link, origin xyz=0 -0.21038 -0.006375 rpy=-1.5708 1.2326E-32 -2.9122E-16, axis 0 0 1, limit lower=-300 upper=300 effort=39 velocity=1.05
- added joint arm_joint_4: type revolute, parent half_arm_2_link, child forearm_link, origin xyz=0 0.006375 -0.21038 rpy=1.5708 -6.6954E-17 -1.6653E-16, axis 0 0 1, limit lower=-2.57 upper=2.57 effort=39 velocity=1.05
- added joint arm_joint_5: type revolute, parent forearm_link, child spherical_wrist_1_link, origin xyz=0 -0.20843 -0.006375 rpy=-1.5708 2.2204E-16 -6.373E-17, axis 0 0 1, limit lower=-300 upper=300 effort=9 velocity=1.05
- added joint arm_joint_6: type revolute, parent spherical_wrist_1_link, child spherical_wrist_2_link, origin xyz=0 0.00017505 -0.10593 rpy=1.5708 9.2076E-28 -8.2157E-15, axis 0 0 1, limit lower=-2.09 upper=2.09 effort=9 velocity=1.05
- added joint arm_joint_7: type revolute, parent spherical_wrist_2_link, child bracelet_link, origin xyz=0 -0.10593 -0.00017505 rpy=-1.5708 -5.5511E-17 9.6396E-17, axis 0 0 1, limit lower=-300 upper=300 effort=9 velocity=1.05
- added joint attachment_to_arm_joint: type fixed, parent attachment, child base_link, origin xyz=0 0 0 rpy=0 0 0, axis 0 0 1
- added joint base_joint_1: type revolute, parent mobile_base_link, child front_left_turning_link, origin xyz=0.1325 -0.13 0.13539 rpy=1.5707963267949 0 0, axis 0 1 0, limit lower=-3.141 upper=3.141 effort=20.0 velocity=0.5
- added joint base_joint_2: type revolute, parent front_left_turning_link, child front_left_caster_link, origin xyz=0.005 -0.08 0.0171140798040203 rpy=0 0 0, axis -1 0 0, limit lower=-300 upper=300 effort=1000 velocity=5.0
- added joint base_joint_3: type revolute, parent mobile_base_link, child front_right_turning_link, origin xyz=-0.1325 -0.13 0.13539 rpy=1.5707963267949 0 0, axis 0 1 0, limit lower=-3.141 upper=3.141 effort=20.0 velocity=0.5
- added joint base_joint_4: type revolute, parent front_right_turning_link, child front_right_caster_link, origin xyz=-0.00500000000000003 -0.08 0.0171140798040204 rpy=0 0 0, axis 1 0 0, limit lower=-300 upper=300 effort=1000 velocity=5.0
- added joint base_joint_5: type revolute, parent mobile_base_link, child back_left_turning_link, origin xyz=0.1325 0.13 0.13539 rpy=1.5707963267949 0 0, axis 0 1 0, limit lower=-3.141 upper=3.141 effort=20.0 velocity=0.5
- added joint base_joint_6: type revolute, parent back_left_turning_link, child back_left_caster_link, origin xyz=0.005 -0.08 -0.0171140798040203 rpy=0 0 0, axis 1 0 0, limit lower=-300 upper=300 effort=1000 velocity=5.0
- added joint base_joint_7: type revolute, parent mobile_base_link, child back_right_turning_link, origin xyz=-0.1325 0.13 0.13539 rpy=1.5707963267949 0 0, axis 0 1 0, limit lower=-3.141 upper=3.141 effort=20.0 velocity=0.5
- added joint base_joint_8: type revolute, parent back_right_turning_link, child back_right_caster_link, origin xyz=-0.005 -0.08 -0.0171140798040203 rpy=0 0 0, axis 1 0 0, limit lower=-300 upper=300 effort=1000 velocity=5.0
- added joint base_to_attachment_joint: type fixed, parent mobile_base_link, child attachment, origin xyz=0 0 0.335 rpy=0 0 3.14159, axis 0 0 1
- added joint root_joint: type fixed, parent root, child mobile_base_link, origin xyz=0 0 0 rpy=0 0 0
